File: KiCad/Capteur_Gaz_SB/Capteur_Gaz_SB/Capteur_Gaz_SB.kicad_pcb (KiCad board)
At the start: 2 copper layers, 68.6 x 53.3 mm, 20 parts, among them P1 Power, P2 Analog, P3 Digital, P4 Digital, P5 CONN_01X01, P6 CONN_01X01, P7 CONN_01X01, P8 CONN_01X01, U1 LTC1050, U2 Capteur_TO-5

Commit message: fin shield SB
Parts:
- added D1: LED, LED_THT:LED_D3.0mm_FlatTop, F.Cu at (173.2, 81.9)
- added J1: Conn_01x02_Female, Connector_Phoenix_MSTB:PhoenixContact_MSTBVA_2,5_2-G-5,08_1x02_P5.08mm_Vertical, F.Cu at (121.2, 84.5)
- added J2: Conn_01x08_Female, Connector_PinSocket_2.54mm:PinSocket_1x08_P2.54mm_Vertical, F.Cu at (170.7, 88.3)
- added Q1: IRF540N, Package_TO_SOT_THT:TO-220-3_Vertical, F.Cu at (135.1, 81.9)
- added R7: 10K, Resistor_THT:R_Axial_DIN0204_L3.6mm_D1.6mm_P7.62mm_Horizontal, F.Cu at (140.2, 81.9)
- added R8: 10K, Resistor_THT:R_Axial_DIN0204_L3.6mm_D1.6mm_P7.62mm_Horizontal, F.Cu at (159.3, 81.9)
- C1, C2, C4: value C -> 100n
- C3: value C -> 1u
- R1: value R -> 10K
- R2: value R -> 100K
- R3: value R -> Rcal1
- R4: value R -> Rcal2
- R5: value R -> 100k
- R6: value R -> 1K
- moved C1 37.0 mm to (126.2, 104.8), turned to 90 degrees
- moved R5 34.1 mm to (142.7, 117.5), turned to 90 degrees
- moved C3 33.2 mm to (138.9, 114.9), turned to 90 degrees
- moved C4 21.0 mm to (161.8, 118.7), turned to 90 degrees
- moved R6 21.0 mm to (158.0, 118.7), turned to 90 degrees
- moved R1 18.7 mm to (122.4, 117.5), turned to 90 degrees
- moved R3 16.8 mm to (133.9, 109.9), turned to 270 degrees
- moved U2 14.6 mm to (121.2, 102.2), turned to 180 degrees
- moved C2 14.4 mm to (159.3, 95.9)
- moved R2 12.5 mm to (126.2, 109.9), turned to 270 degrees
- moved U1 9.32 mm to (147.8, 93.3)
- moved R4 4.00 mm to (130.0, 117.5), turned to 90 degrees
Connections:
- P2 pad 1: /A0 -> ANx_Arduino
- U2 pad 1: +3V3 -> Net-(J1-Pad2)
- U2 pad 2: GND -> Net-(Q1-Pad2)
- U2 pad 3: Net-(U2-Pad3) -> +3V3
Routing:
- net +3V3: track 0.00 -> 99.2 mm, vias 0 -> 2
- net /13(SCK): track 0.00 -> 48.4 mm, vias 0 -> 2
- net Net-(C3-Pad1): track 0.00 -> 40.6 mm, vias 0 -> 2
- net /12(MISO): track 0.00 -> 39.3 mm, vias 0 -> 2
- net +5V: track 0.00 -> 35.9 mm
- net /11(**/MOSI): track 0.00 -> 35.2 mm, vias 0 -> 2
- net /4: track 0.00 -> 34.7 mm
- net Net-(C1-Pad1): track 0.00 -> 33.1 mm
- net Net-(Q1-Pad2): track 0.00 -> 31.7 mm, vias 0 -> 2
- net Net-(C3-Pad2): track 0.00 -> 28.0 mm, vias 0 -> 2
- net Net-(R1-Pad1): track 0.00 -> 22.6 mm
- net Net-(J1-Pad2): track 0.00 -> 12.7 mm
- net ANx_Arduino: track 0.00 -> 8.89 mm
- net Net-(R3-Pad2): track 0.00 -> 3.81 mm
- net Net-(D1-Pad2): track 0.00 -> 3.81 mm
