File: KiCad/Capteur_Gaz_SB/Capteur_Gaz_SB/Capteur_Gaz_SB.sch (KiCad schematic (older format))
At the start: 25 parts, among them J1 Conn_01x02_Female, P1 Power, P2 Analog, P3 Digital, P4 Digital, P5 CONN_01X01, P6 CONN_01X01, P7 CONN_01X01, P8 CONN_01X01, Q1 IRF540N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

Commit message: fin shield SB
Parts:
- added J2: Conn_01x08_Female, Connector_PinSocket_2.54mm:PinSocket_1x08_P2.54mm_Vertical, symbol Connector:Conn_01x08_Female
- U1: symbol LTC1050:LTC1050 -> Capteur_Gaz_SB-rescue:LTC1050-LTC1050
- U2: symbol LTC1050:Capteur_TO-5 -> Capteur_Gaz_SB-rescue:Capteur_TO-5-LTC1050
Connections:
- net +3V3: now also J2.6 (Pin_6)
- net 11(**/MOSI): now also J2.1 (Pin_1)
- net 12(MISO): now also J2.2 (Pin_2)
- net 13(SCK): now also J2.5 (Pin_5)
- net 4: now also P4.4 (Pin_4)
- net GND: now also J2.8 (Pin_8)
- no-connect marks 7 -> 10
Other:
- moved on the sheet: C1, C2, C3, C4, D1, J1, Q1, R1, R2, R3, R4, R5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

Commit message: modification et ajout carte pour capteur en salle blanche
Connections:
- no-connect marks 10 -> 11
Changed lines of the file:
@@
 	8950 2300 8950 1450
 Wire Wire Line
-	9050 2000 9050 1350
-Wire Wire Line
-	9150 1900 9150 1450
+	9050 2000 9050 1400
+Wire Wire Line
+	9150 1900 9150 1500
 Wire Wire Line
 	9400 2500 8900 2500
@@
 	9300 2100 9300 2200
 Wire Wire Line
-	9300 2200 9300 3150
+	9300 2200 9300 3100
 Wire Notes Line
 	8500 500  8500 3450
@@
 Text Label 3650 2150 2    60   ~ 0
 13(SCK)
+$Comp
+L power:PWR_FLAG #FLG0101
+U 1 1 5BE16F3A
+P 8650 1100
+F 0 "#FLG0101" H 8650 1175 50  0001 C CNN
+F 1 "PWR_FLAG" H 8650 1274 50  0000 C CNN
+F 2 "" H 8650 1100 50  0001 C CNN
+F 3 "~" H 8650 1100 50  0001 C CNN
+	1    8650 1100
+	1    0    0    -1
+$EndComp
+$Comp
+L power:PWR_FLAG #FLG0102
+U 1 1 5BE16F90
+P 9250 1050
+F 0 "#FLG0102" H 9250 1125 50  0001 C CNN
+F 1 "PWR_FLAG" H 9250 1224 50  0000 C CNN
+F 2 "" H 9250 1050 50  0001 C CNN
+F 3 "~" H 9250 1050 50  0001 C CNN
+	1    9250 1050
+	1    0    0    -1
+$EndComp
+Wire Wire Line
+	9150 1500 9250 1500
+Wire Wire Line
+	9250 1500 9250 1050
+Connection ~ 9150 1500
+Wire Wire Line
+	9150 1500 9150 1450
+Wire Wire Line
+	9050 1400 8650 1400
+Wire Wire Line
+	8650 1400 8650 1100
+Connection ~ 9050 1400
+Wire Wire Line
+	9050 1400 9050 1350
+$Comp
+L power:PWR_FLAG #FLG0103
+U 1 1 5BE1BF2D
+P 8900 3200
+F 0 "#FLG0103" H 8900 3275 50  0001 C CNN
+F 1 "PWR_FLAG" H 8900 3374 50  0000 C CNN
+F 2 "" H 8900 3200 50  0001 C CNN
+F 3 "~" H 8900 3200 50  0001 C CNN
+	1    8900 3200
+	0    -1   -1   0
+$EndComp
+Wire Wire Line
+	9300 3100 8900 3100
+Wire Wire Line
+	8900 3100 8900 3200
+Connection ~ 9300 3100
+Wire Wire Line
+	9300 3100 9300 3150
+NoConn ~ 4750 5150
 $EndSCHEMATC
